Commit message: Updated core URDF

File: description/robot_core.xacro (robot description, xacro)
@@ -21,29 +21,29 @@
         <parent link="base_link"/>
         <child link="chassis"/>
-        <origin xyz="0.1 0 0"/>
+        <origin xyz="-0.1 0 0"/>
     </joint>
     <link name="chassis">
         <visual>
-            <origin xyz="0.06 0 0.075"/>
+            <origin xyz="0.13 0 0.032"/>
             <geometry>
-                <box size="0.3 0.3 0.15"/>
+                <box size="0.26 0.152 0.063"/>
             </geometry>
             <material name="white"/>
         </visual>
          <collision>
-            <origin xyz="0.06 0 0.075"/>
+            <origin xyz="0.13 0 0.032"/>
             <geometry>
-                <box size="0.3 0.3 0.15"/>
+                <box size="0.26 0.152 0.063"/>
             </geometry>
         </collision>
-        <xacro:inertial_box mass="0.5" x="0.3" y="0.3" z="0.15">
-            <origin xyz="0.06 0 0.075"/>
+        <xacro:inertial_box mass="0.5" x="0.26" y="0.152" z="0.063">
+            <origin xyz="0.13 0 0.032" rpy="0 0 0"/>
         </xacro:inertial_box>
     </link>
 <!--  left wheel link-->
     <joint name="left_wheel_joint" type="continuous">
-        <parent link="chassis"/>
+        <parent link="base_link"/>
         <child link="left_wheel"/>
-        <origin xyz="0 0.175 0" rpy="-${pi/2} 0 0"/>
+        <origin xyz="0 0.1 0" rpy="-${pi/2} 0 0"/>
         <axis xyz="0 0 1" />
     </joint>
@@ -66,7 +66,7 @@
 <!--  right wheel link-->
     <joint name="right_wheel_joint" type="continuous">
-        <parent link="chassis"/>
+        <parent link="base_link"/>
         <child link="right_wheel"/>
-        <origin xyz="0 -0.175 0" rpy="${pi/2} 0 0"/>
+        <origin xyz="0 -0.1 0" rpy="${pi/2} 0 0"/>
         <axis xyz="0 0 -1" />
     </joint>
@@ -91,5 +91,5 @@
         <parent link="chassis"/>
         <child link="center_wheel"/>
-        <origin xyz="0.16 0 0" />
+        <origin xyz="0.2 0 0" />
     </joint>
     <link name="center_wheel">
@@ -106,5 +106,5 @@
         </collision>
         <xacro:inertial_sphere mass="0.1" radius="0.05">
-            <origin xyz="0 0 0" rpy="0 0 0"/>
+            <origin xyz="0.2 0 0" rpy="0 0 0"/>
         </xacro:inertial_sphere>
     </link>
